Commit message: Added armsgit add .git add .git add ./usr/bin/python3 -m pip install ipykernel torch --break-system-packages  Full body complete

File: rpo_description/models/full_robot/urdf/full_robot.urdf (robot description, URDF)
Before this commit: robot full_robot, 96 links, 95 joints
Links:
- added link arm_link, mass 0.156428; visual mesh filename=package://rpo_description/models/full_robot/meshes/Arm_Link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 scale=1 1 1
- added link arm_link_1, mass 0.156428; visual mesh filename=package://rpo_description/models/full_robot/meshes/Arm_Link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 scale=1 1 1
- added link arm_link_2, mass 0.156428; visual mesh filename=package://rpo_description/models/full_robot/meshes/Arm_Link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 scale=1 1 1
- added link arm_link_3, mass 0.156428; visual mesh filename=package://rpo_description/models/full_robot/meshes/Arm_Link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 scale=1 1 1
- added link dm_j4340_controller_cover_10, mass 0.0142077; visual mesh filename=package://rpo_description/models/full_robot/meshes/DM_J4340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 scale=1 1 1
- added link dm_j4340_controller_cover_11, mass 0.0142077; visual mesh filename=package://rpo_description/models/full_robot/meshes/DM_J4340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 scale=1 1 1
- added link dm_j4340_controller_cover_12, mass 0.0142077; visual mesh filename=package://rpo_description/models/full_robot/meshes/DM_J4340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 scale=1 1 1
- added link dm_j4340_controller_cover_13, mass 0.0142077; visual mesh filename=package://rpo_description/models/full_robot/meshes/DM_J4340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 scale=1 1 1
- added link dm_j4340_controller_cover_6, mass 0.0142077; visual mesh filename=package://rpo_description/models/full_robot/meshes/DM_J4340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 scale=1 1 1
- added link dm_j4340_controller_cover_7, mass 0.0142077; visual mesh filename=package://rpo_description/models/full_robot/meshes/DM_J4340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 scale=1 1 1
- added link dm_j4340_controller_cover_8, mass 0.0142077; visual mesh filename=package://rpo_description/models/full_robot/meshes/DM_J4340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 scale=1 1 1
- added link dm_j4340_controller_cover_9, mass 0.0142077; visual mesh filename=package://rpo_description/models/full_robot/meshes/DM_J4340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 scale=1 1 1
- added link dm_j4340_motor_10, mass 0.995728; visual mesh filename=package://rpo_description/models/full_robot/meshes/DM_J4340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 scale=1 1 1
- added link dm_j4340_motor_11, mass 0.995728; visual mesh filename=package://rpo_description/models/full_robot/meshes/DM_J4340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 scale=1 1 1
- added link dm_j4340_motor_12, mass 0.995728; visual mesh filename=package://rpo_description/models/full_robot/meshes/DM_J4340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 scale=1 1 1
- added link dm_j4340_motor_13, mass 0.995728; visual mesh filename=package://rpo_description/models/full_robot/meshes/DM_J4340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 scale=1 1 1
- added link dm_j4340_motor_6, mass 0.995728; visual mesh filename=package://rpo_description/models/full_robot/meshes/DM_J4340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 scale=1 1 1
- added link dm_j4340_motor_7, mass 0.995728; visual mesh filename=package://rpo_description/models/full_robot/meshes/DM_J4340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 scale=1 1 1
- added link dm_j4340_motor_8, mass 0.995728; visual mesh filename=package://rpo_description/models/full_robot/meshes/DM_J4340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 scale=1 1 1
- added link dm_j4340_motor_9, mass 0.995728; visual mesh filename=package://rpo_description/models/full_robot/meshes/DM_J4340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 scale=1 1 1
- added link end_cap, mass 0.134915; visual mesh filename=package://rpo_description/models/full_robot/meshes/End_Cap.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 scale=1 1 1
- added link end_cap_1, mass 0.134915; visual mesh filename=package://rpo_description/models/full_robot/meshes/End_Cap.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 scale=1 1 1
- added link end_cap_2, mass 0.134915; visual mesh filename=package://rpo_description/models/full_robot/meshes/End_Cap.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 scale=1 1 1
- added link end_cap_3, mass 0.134915; visual mesh filename=package://rpo_description/models/full_robot/meshes/End_Cap.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 scale=1 1 1
- added link shoulder_bracket_a, mass 0.0829317; visual mesh filename=package://rpo_description/models/full_robot/meshes/Shoulder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 scale=1 1 1
- added link shoulder_bracket_a_1, mass 0.0829317; visual mesh filename=package://rpo_description/models/full_robot/meshes/Shoulder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 scale=1 1 1
- added link shoulder_bracket_a_2, mass 0.0829317; visual mesh filename=package://rpo_description/models/full_robot/meshes/Shoulder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 scale=1 1 1
- added link shoulder_bracket_a_3, mass 0.0829317; visual mesh filename=package://rpo_description/models/full_robot/meshes/Shoulder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 scale=1 1 1
- added link shoulder_bracket_b, mass 0.0758319; visual mesh filename=package://rpo_description/models/full_robot/meshes/Shoulder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 scale=1 1 1
- added link shoulder_bracket_b_1, mass 0.0758319; visual mesh filename=package://rpo_description/models/full_robot/meshes/Shoulder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 scale=1 1 1
- added link shoulder_bracket_b_2, mass 0.0758319; visual mesh filename=package://rpo_description/models/full_robot/meshes/Shoulder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 scale=1 1 1
- added link shoulder_bracket_b_3, mass 0.0758319; visual mesh filename=package://rpo_description/models/full_robot/meshes/Shoulder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 scale=1 1 1
Joints:
- added joint fastened_3_4: type fixed, parent hip_plate, child hip_plate_1, origin xyz=-1.06443e-14 0.063 -0.023 rpy=-5.91202e-34 -8.29804e-17 1.42492e-17, axis -1 0 0
- added joint fastened_3_5: type fixed, parent shoulder_bracket_a_2, child dm_j4340_motor_6, origin xyz=0.056 0 0.01825 rpy=-1.5708 -1.11022e-16 -1.5708, axis 0 -1 0
- added joint fastened_4_4: type fixed, parent hip_connector_a, child dm_j10010l_rotor_4, origin xyz=-5.55112e-17 0.02385 0.0715 rpy=8.23639e-47 -8.32667e-17 -1.97832e-30, axis 0 -1 -1.19142e-27
- added joint fastened_4_5: type fixed, parent dm_j4340_motor_7, child arm_link_3, origin xyz=-3.46945e-18 0.00175 -2.77556e-17 rpy=3.14159 0.000118363 -7.88937e-31, axis -0 -1 -0
- added joint fastened_5_4: type fixed, parent hip_connector_a_3, child dm_j10010l_stator__1_, origin xyz=1.38778e-17 0.02385 0.0715 rpy=1.94289e-16 3.96948e-17 7.85687e-17, axis 0 1 1.19142e-27
- added joint fastened_5_5: type fixed, parent arm_link_3, child end_cap_2, origin xyz=-1.73472e-17 -0.117 -2.77556e-17 rpy=-9.86076e-31 0 0, axis 0 1 0
- added joint fastened_6_4: type fixed, parent dm_j10010l_stator__1_, child hip_connector_b_1, origin xyz=0.0428779 -0.0377 0.0311526 rpy=-1.5708 3.10311e-16 3.14159, axis 0 0 -1
- added joint fastened_6_5: type fixed, parent end_cap_2, child shoulder_bracket_a_3, origin xyz=0 -0.013 5.55112e-17 rpy=3.14159 1.90742e-30 -1.5708, axis -1 0 0
- added joint fastened_7_4: type fixed, parent dm_j10010l_rotor_4, child hip_connector_b_2, origin xyz=-0.0428779 -0.0372 0.0311526 rpy=-1.5708 -5.58745e-16 -3.14159, axis 0 0 -1
- added joint fastened_7_5: type fixed, parent shoulder_bracket_a_3, child dm_j4340_motor_5, origin xyz=0.056 -3.46945e-18 0.01825 rpy=-1.5708 -0 -1.5708, axis 0 -1 0
- added joint fastened_8_2: type fixed, parent dm_j4340_motor_4, child arm_link_2, origin xyz=0 0.00175 0 rpy=3.14159 -3.15544e-30 -7.88861e-30, axis -0 -1 -0
- added joint fastened_8_3: type fixed, parent end_cap, child shoulder_bracket_a, origin xyz=0 -0.014 3.46945e-18 rpy=-1.5708 -0 -1.5708, axis -1 0 0
- added joint fastened_9_2: type fixed, parent hip_connector_a_2, child dm_j10010l_stator__2_, origin xyz=6.93889e-17 0.01985 0.0715 rpy=0 1.5708 2.28976e-15, axis 0 1 1.19142e-27
- added joint fastened_9_3: type fixed, parent arm_link_2, child end_cap_3, origin xyz=0 -0.117 0 rpy=-8.87469e-31 0 0, axis 0 1 0
- added joint group_1_fastened_joint_18: type fixed, parent dm_j10010l_stator__1_, child dm_j10010l_rotor_7, origin xyz=0 0.0277355 -1.77358e-14 rpy=-6.0831e-64 1.92593e-32 -6.31705e-32, axis -0 -0 -1
- added joint group_1_fastened_joint_19: type fixed, parent dm_j10010l_rotor_7, child dm_j10010l_side_cover_5, origin xyz=-1.38778e-17 1.38778e-17 0 rpy=-6.0831e-64 1.92593e-32 -6.31705e-32, axis -0 -0 -1
- added joint group_1_fastened_joint_20: type fixed, parent dm_j10010l_side_cover_5, child dm_j10010l_controller_cover_4, origin xyz=-1.38778e-17 1.38778e-17 0 rpy=-6.0831e-64 1.92593e-32 -6.31705e-32, axis -0 -0 -1
- added joint group_1_fastened_joint_21: type fixed, parent dm_j4340_motor_1, child dm_j4340_controller_cover_1, origin xyz=2.77556e-17 0 -3.46945e-18 rpy=3.34096e-52 -6.77626e-21 -9.86076e-32, axis 0 0 1
- added joint group_1_fastened_joint_22: type fixed, parent dm_j4340_motor_4, child dm_j4340_controller_cover_4, origin xyz=0 1.38778e-17 0 rpy=-3.36312e-44 0 0, axis 0 0 1
- added joint group_1_fastened_joint_23: type fixed, parent dm_j4340_motor_7, child dm_j4340_controller_cover_7, origin xyz=0 0 -2.77556e-17 rpy=-4.66859e-35 0.000118363 -7.88861e-31, axis 0 0 1
- added joint group_1_fastened_joint_24: type fixed, parent dm_j4340_motor_5, child dm_j4340_controller_cover_5, origin xyz=0 -0.00175 0 rpy=0 0 -1.2962e-44, axis 0 0 1
- added joint group_1_fastened_joint_25: type fixed, parent dm_j4340_motor_6, child dm_j4340_controller_cover_6, origin xyz=-5.55112e-17 -0.00175 0 rpy=7.00649e-46 -0 0, axis 0 0 1
- added joint left_elbow_joint: type revolute, parent dm_j4340_motor, child shoulder_bracket_b, origin xyz=-6.93889e-18 -0.00175 0 rpy=0 -1.5708 1.5708, axis 0 0 1, limit lower=-0.6 upper=1.57 effort=27 velocity=8
- added joint left_shoulder_pitch_joint: type revolute, parent dm_j4340_motor_8, child shoulder_bracket_a_1, origin xyz=0 -0.00175 -3.88578e-16 rpy=1.5708 -0 -1.5708, axis 1 0 0, limit lower=-3.14 upper=1.57 effort=27 velocity=8
- added joint left_shoulder_roll_joint: type revolute, parent dm_j4340_motor_3, child shoulder_bracket_b_3, origin xyz=-2.77556e-17 -0.00175 -5.55112e-17 rpy=1.5708 -5.5434e-25 9.74653e-24, axis 0 0 1, limit lower=-0.25 upper=3.14 effort=27 velocity=8
- added joint left_shoulder_yaw_joint: type revolute, parent shoulder_bracket_b_3, child dm_j4340_motor_1, origin xyz=0 -0.049 -0.02 rpy=-3.14159 6.77626e-21 9.86076e-32, axis 0 1 0, limit lower=-1.57 upper=1.57 effort=27 velocity=8
- added joint left_wrist_roll_joint: type revolute, parent shoulder_bracket_b, child dm_j4340_motor_2, origin xyz=-4.16334e-17 -0.05 -0.02 rpy=0 -1.5708 3.14159, axis 0 1 0, limit lower=-1.57 upper=1.57 effort=27 velocity=8
- added joint right_elbow_joint: type revolute, parent dm_j4340_motor_5, child shoulder_bracket_b_2, origin xyz=0 -0.00175 -6.93889e-18 rpy=0 1.5708 4.71239, axis 0 0 -1, limit lower=-0.6 upper=1.57 effort=27 velocity=8
- added joint right_shoulder_pitch_joint: type revolute, parent dm_j4340_motor_9, child shoulder_bracket_a_2, origin xyz=-1.38778e-17 -0.00175 0 rpy=1.5708 -0 -1.5708, axis -1 0 0, limit lower=-3.14 upper=1.57 effort=27 velocity=8
- added joint right_shoulder_roll_joint: type revolute, parent dm_j4340_motor_6, child shoulder_bracket_b_1, origin xyz=-5.55112e-17 -0.00175 2.77556e-17 rpy=0 1.5708 -1.5708, axis 0 0 1, limit lower=-3.14 upper=0.25 effort=27 velocity=8
- added joint right_shoulder_yaw_joint: type revolute, parent shoulder_bracket_b_1, child dm_j4340_motor_7, origin xyz=0 -0.05 -0.02 rpy=0 1.5708 -3.14159, axis 0 1 0, limit lower=-1.57 upper=1.57 effort=27 velocity=8
- added joint right_wrist_roll_joint: type revolute, parent shoulder_bracket_b_2, child dm_j4340_motor_4, origin xyz=0 -0.05 -0.02 rpy=-1.61716e-29 4.71344e-29 -3.14159, axis 0 1 0, limit lower=-1.57 upper=1.57 effort=27 velocity=8
- joint fastened_1: child dm_j10010l_stator__1__1 -> dm_j10010l_stator__1__4
- joint fastened_10: child dm_j4340_motor -> dm_j4340_motor_8
- joint fastened_11: child dm_j4340_motor_1 -> dm_j4340_motor_9; origin xyz=0.0195 0.0625 -1.84575e-15 rpy=-1.5708 -0 -1.5708 -> xyz=0.0195 0.0625 0 rpy=-1.5708 -0 -1.5708
- joint fastened_12: parent dm_j4340_motor_4 -> dm_j4340_motor_12
- joint fastened_12_1: parent dm_j4340_motor_3 -> dm_j4340_motor_11
- joint fastened_2_1: child dm_j10010l_rotor_8 -> dm_j10010l_rotor_2
- joint fastened_2_3: child dm_j10010l_rotor_5 -> dm_j10010l_rotor_6
- joint fastened_3_1: child dm_j4340_motor_5 -> dm_j4340_motor_3; origin xyz=3.36883e-15 -0.19 -0.0005 rpy=-1.5708 4.44089e-16 1.5708 -> xyz=0.056 -3.77476e-15 0.01825 rpy=-1.5708 -6.77626e-21 -6.77626e-21; parent lower_leg_1 -> shoulder_bracket_a_1
- joint fastened_3_2: child dm_j4340_motor_2 -> dm_j4340_motor_13; origin xyz=3.48159e-15 -0.19 -0.0005 rpy=-1.5708 -1.55431e-15 1.5708 -> xyz=3.36883e-15 -0.19 -0.0005 rpy=-1.5708 4.44089e-16 1.5708; parent lower_leg -> lower_leg_1
- joint fastened_3_3: axis -1 0 0 -> 0 -1 0; child hip_plate_1 -> dm_j4340_motor_10; origin xyz=-1.06443e-14 0.063 -0.023 rpy=-5.91202e-34 -8.29804e-17 1.42492e-17 -> xyz=3.48159e-15 -0.19 -0.0005 rpy=-1.5708 -1.55431e-15 1.5708; parent hip_plate -> lower_leg
- joint fastened_4: origin xyz=-0.0605 -0.06 0.0085 rpy=0 -1.5708 -3.88434e-33 -> xyz=-0.0604929 -0.0600072 0.0085 rpy=0 -1.5708 0.000118363
- joint fastened_4_1: axis 0 -1 0 -> -0 -1 -0; child dm_j4340_motor_4 -> arm_link; origin xyz=3.35496e-15 -0.12 -0.0005 rpy=-1.5708 4.44089e-16 1.5708 -> xyz=-5.55112e-17 0.00175 -2.08167e-17 rpy=-3.14159 5.2638e-20 -1.1189e-16; parent lower_leg_1 -> dm_j4340_motor_2
- joint fastened_4_2: child dm_j4340_motor_3 -> dm_j4340_motor_12; origin xyz=3.42781e-15 -0.12 -0.0005 rpy=-1.5708 7.77156e-16 1.5708 -> xyz=3.35496e-15 -0.12 -0.0005 rpy=-1.5708 4.44089e-16 1.5708; parent lower_leg -> lower_leg_1
- joint fastened_4_3: axis 0 -1 -1.19142e-27 -> 0 -1 0; child dm_j10010l_rotor_3 -> dm_j4340_motor_11; origin xyz=-5.55112e-17 0.02385 0.0715 rpy=8.23639e-47 -8.32667e-17 -1.97832e-30 -> xyz=3.42781e-15 -0.12 -0.0005 rpy=-1.5708 7.77156e-16 1.5708; parent hip_connector_a -> lower_leg
- joint fastened_5: origin xyz=0.0605 0.06 0.0085 rpy=0 1.5708 -1.04329e-16 -> xyz=0.0604929 0.0600072 0.0085 rpy=0 1.5708 0.000118363
- joint fastened_5_1: axis 0 1 0 -> -0 -1 -0; child calf_bearing_lock_2 -> arm_link_1; origin xyz=-0.0065 -0.289 0.002575 rpy=-1.5708 -2.46646e-17 3.14159 -> xyz=-5.55112e-17 0.00175 1.38778e-17 rpy=3.14159 -1.35525e-20 -9.87061e-21; parent lower_leg_1 -> dm_j4340_motor_1
- joint fastened_5_2: child calf_bearing_lock_1 -> calf_bearing_lock_2; origin xyz=-0.0065 -0.289 0.002575 rpy=-1.5708 5.25226e-16 -3.14159 -> xyz=-0.0065 -0.289 0.002575 rpy=-1.5708 -2.46646e-17 3.14159; parent lower_leg -> lower_leg_1
- joint fastened_5_3: axis 0 1 1.19142e-27 -> 0 1 0; child dm_j10010l_stator__1_ -> calf_bearing_lock_1; origin xyz=1.38778e-17 0.02385 0.0715 rpy=1.94289e-16 3.96948e-17 7.85687e-17 -> xyz=-0.0065 -0.289 0.002575 rpy=-1.5708 5.25226e-16 -3.14159; parent hip_connector_a_3 -> lower_leg
- joint fastened_6_1: child calf_bearing_lock_3 -> end_cap_1; origin xyz=-0.0065 -0.289 -0.041275 rpy=1.5708 2.81655e-18 2.38762e-18 -> xyz=5.55112e-17 -0.1175 1.04083e-16 rpy=-1.57772e-30 1.06911e-50 1.35525e-20; parent lower_leg_1 -> arm_link
- joint fastened_6_2: child calf_bearing_lock -> calf_bearing_lock_3; origin xyz=-0.0065 -0.289 -0.041275 rpy=1.5708 5.81376e-16 6.36248e-16 -> xyz=-0.0065 -0.289 -0.041275 rpy=1.5708 2.81655e-18 2.38762e-18; parent lower_leg -> lower_leg_1
- joint fastened_6_3: axis 0 0 -1 -> 0 1 0; child hip_connector_b_1 -> calf_bearing_lock; origin xyz=0.0428779 -0.0377 0.0311526 rpy=-1.5708 3.10311e-16 3.14159 -> xyz=-0.0065 -0.289 -0.041275 rpy=1.5708 5.81376e-16 6.36248e-16; parent dm_j10010l_stator__1_ -> lower_leg
- joint fastened_7: axis 0 0 -1 -> 0 1 0; child torso_shoulder_bracket -> end_cap; origin xyz=-0.218676 0.06 0.002 rpy=-1.5708 -5.10251e-18 -8.31764e-16 -> xyz=1.11022e-16 -0.1165 2.70617e-16 rpy=4.84861e-25 2.64856e-35 -8.0245e-25; parent torso_back_plate -> arm_link_1
- joint fastened_7_1: axis -1 -0 -0 -> 0 0 -1; child ankle_roll_connector_2 -> torso_shoulder_bracket; origin xyz=0.062 -0.0135 -1.11022e-16 rpy=0 1.5708 1.17845e-27 -> xyz=-0.218676 0.06 0.002 rpy=-1.5708 -5.10251e-18 -8.31764e-16; parent foot_1 -> torso_back_plate
- joint fastened_7_2: axis 0 0 -1 -> -1 -0 -0; child foot -> ankle_roll_connector_2; origin xyz=-0.03 2.77556e-17 0.011 rpy=0 -1.5708 5.42238e-27 -> xyz=0.062 -0.0135 -1.11022e-16 rpy=0 1.5708 1.17845e-27; parent ankle_roll_connector_1 -> foot_1
- joint fastened_7_3: child hip_connector_b_2 -> foot; origin xyz=-0.0428779 -0.0372 0.0311526 rpy=-1.5708 -5.58745e-16 -3.14159 -> xyz=-0.03 2.77556e-17 0.011 rpy=0 -1.5708 5.42238e-27; parent dm_j10010l_rotor_3 -> ankle_roll_connector_1
- joint fastened_9: axis 0 0 -1 -> 0 -1 0; child torso_side_plate_1 -> dm_j4340_motor; origin xyz=-0.013 -0.133 0.002 rpy=0 -1.5708 1.5708 -> xyz=0.056 1.14492e-16 0.01825 rpy=-1.5708 1.11022e-16 -1.5708; parent torso_back_plate -> shoulder_bracket_a
- joint fastened_9_1: axis 0 1 1.19142e-27 -> 0 0 -1; child dm_j10010l_stator__2_ -> torso_side_plate_1; origin xyz=6.93889e-17 0.01985 0.0715 rpy=0 1.5708 2.28976e-15 -> xyz=-0.013 -0.133 0.002 rpy=0 -1.5708 1.5708; parent hip_connector_a_2 -> torso_back_plate
- joint group_1__1__fastened_joint: child dm_j10010l_side_cover_7 -> dm_j10010l_side_cover_8; parent dm_j10010l_rotor_7 -> dm_j10010l_rotor_8
- joint group_1__1__fastened_joint_1: child dm_j10010l_controller_cover_6 -> dm_j10010l_controller_cover_7; parent dm_j10010l_side_cover_7 -> dm_j10010l_side_cover_8
- joint group_1__1__fastened_joint_2: child dm_j10010l_rotor_7 -> dm_j10010l_rotor_8
- joint group_1__2__fastened_joint: child dm_j10010l_side_cover_3 -> dm_j10010l_side_cover_4; parent dm_j10010l_rotor_2 -> dm_j10010l_rotor_3
- joint group_1__2__fastened_joint_1: child dm_j10010l_rotor_2 -> dm_j10010l_rotor_3
- joint group_1__2__fastened_joint_2: child dm_j10010l_controller_cover_2 -> dm_j10010l_controller_cover_3; parent dm_j10010l_side_cover_3 -> dm_j10010l_side_cover_4
- joint group_1__3__fastened_joint: parent dm_j10010l_rotor_3 -> dm_j10010l_rotor_4
- joint group_1__3__fastened_joint_1: child dm_j10010l_controller_cover_5 -> dm_j10010l_controller_cover_6; parent dm_j10010l_side_cover_5 -> dm_j10010l_side_cover_6
- joint group_1__3__fastened_joint_2: child dm_j10010l_side_cover_5 -> dm_j10010l_side_cover_6
- joint group_1__4__fastened_joint: child dm_j10010l_controller_cover_4 -> dm_j10010l_controller_cover_5; parent dm_j10010l_side_cover_2 -> dm_j10010l_side_cover_3
- joint group_1__4__fastened_joint_1: child dm_j10010l_side_cover_2 -> dm_j10010l_side_cover_3
- joint group_1__4__fastened_joint_2: parent dm_j10010l_rotor_5 -> dm_j10010l_rotor_6
- joint group_1__5__fastened_joint: child dm_j10010l_rotor_4 -> dm_j10010l_rotor_5
- joint group_1__5__fastened_joint_1: child dm_j10010l_side_cover_6 -> dm_j10010l_side_cover_7; parent dm_j10010l_rotor_4 -> dm_j10010l_rotor_5
- joint group_1__5__fastened_joint_2: child dm_j10010l_controller_cover_7 -> dm_j10010l_controller_cover_8; parent dm_j10010l_side_cover_6 -> dm_j10010l_side_cover_7
- joint group_1_fastened_joint: origin xyz=-3.46945e-18 -0.00175 0 rpy=0 -0 7.00649e-46 -> xyz=0 -0.00175 6.93889e-18 rpy=-9.86076e-32 7.88861e-31 6.77626e-21
- joint group_1_fastened_joint_1: axis -0 -0 -1 -> 0 0 1; child dm_j10010l_rotor -> dm_j4340_controller_cover_8; origin xyz=0 0.0277355 -1.77636e-14 rpy=2.46519e-32 -8.59206e-33 -3.9443e-31 -> xyz=-6.93889e-18 -0.00175 0 rpy=0 0 -1.53101e-37; parent dm_j10010l_stator__1__1 -> dm_j4340_motor_8
- joint group_1_fastened_joint_10: axis 0 0 1 -> -0 -0 -1; child dm_j4340_controller_cover_2 -> dm_j10010l_side_cover_2; origin xyz=1.11022e-16 -0.00025 1.73472e-18 rpy=6.24836e-33 3.9443e-31 1.23227e-63 -> xyz=-1.73472e-18 0.0659355 5.55112e-17 rpy=1.2326e-32 1.70026e-74 -2.75883e-42; parent dm_j4340_motor_2 -> dm_j10010l_rotor_2
- joint group_1_fastened_joint_11: axis 0 0 1 -> -0 -0 -1; child dm_j10010l_stator__1__4 -> dm_j10010l_controller_cover_2; origin xyz=0 0.0659355 0 rpy=0 -0 7.00649e-46 -> xyz=-1.73472e-18 -3.46945e-18 5.55112e-17 rpy=1.2326e-32 1.70026e-74 -2.75883e-42; parent dm_j10010l_rotor_1 -> dm_j10010l_side_cover_2
- joint group_1_fastened_joint_12: axis -0 -0 -1 -> 0 0 1; child dm_j10010l_side_cover_1 -> dm_j4340_controller_cover_12; origin xyz=0 0.0659355 0 rpy=0 -0 7.00649e-46 -> xyz=1.11022e-16 -0.00025 0 rpy=1.50704e-32 -0 0; parent dm_j10010l_rotor_1 -> dm_j4340_motor_12
- joint group_1_fastened_joint_13: axis -0 -0 -1 -> 0 0 1; child dm_j10010l_controller_cover_1 -> dm_j4340_controller_cover_10; origin xyz=-1.73472e-18 0 -5.55112e-17 rpy=0 -0 7.00649e-46 -> xyz=1.11022e-16 -0.00025 1.73472e-18 rpy=6.24836e-33 3.9443e-31 1.23227e-63; parent dm_j10010l_side_cover_1 -> dm_j4340_motor_10
- joint group_1_fastened_joint_14: child dm_j4340_controller_cover_3 -> dm_j10010l_stator__1__1; origin xyz=1.11022e-16 -0.00025 -1.73472e-18 rpy=-2.53841e-32 5.00613e-63 3.9443e-31 -> xyz=0 0.0659355 0 rpy=0 -0 7.00649e-46; parent dm_j4340_motor_3 -> dm_j10010l_rotor_1
- joint group_1_fastened_joint_15: child dm_j10010l_rotor_6 -> dm_j10010l_side_cover_1; origin xyz=0 0.0277355 -1.77358e-14 rpy=-6.0831e-64 1.92593e-32 -6.31705e-32 -> xyz=0 0.0659355 0 rpy=0 -0 7.00649e-46; parent dm_j10010l_stator__1_ -> dm_j10010l_rotor_1
- joint group_1_fastened_joint_16: child dm_j10010l_side_cover_4 -> dm_j10010l_controller_cover_1; origin xyz=-1.38778e-17 1.38778e-17 0 rpy=-6.0831e-64 1.92593e-32 -6.31705e-32 -> xyz=-1.73472e-18 0 -5.55112e-17 rpy=0 -0 7.00649e-46; parent dm_j10010l_rotor_6 -> dm_j10010l_side_cover_1
- joint group_1_fastened_joint_17: axis -0 -0 -1 -> 0 0 1; child dm_j10010l_controller_cover_3 -> dm_j4340_controller_cover_11; origin xyz=-1.38778e-17 1.38778e-17 0 rpy=-6.0831e-64 1.92593e-32 -6.31705e-32 -> xyz=1.11022e-16 -0.00025 -1.73472e-18 rpy=-2.53841e-32 5.00613e-63 3.9443e-31; parent dm_j10010l_side_cover_4 -> dm_j4340_motor_11
- joint group_1_fastened_joint_2: child dm_j10010l_side_cover -> dm_j10010l_rotor; origin xyz=0 0 0 rpy=2.46519e-32 -8.59206e-33 -3.9443e-31 -> xyz=0 0.0277355 -1.77636e-14 rpy=2.46519e-32 -8.59206e-33 -3.9443e-31; parent dm_j10010l_rotor -> dm_j10010l_stator__1__4
- joint group_1_fastened_joint_3: child dm_j10010l_controller_cover -> dm_j10010l_side_cover; parent dm_j10010l_side_cover -> dm_j10010l_rotor
- joint group_1_fastened_joint_4: axis 0 0 1 -> -0 -0 -1; child dm_j4340_controller_cover_1 -> dm_j10010l_controller_cover; origin xyz=0 -0.00175 0 rpy=0 -0 0 -> xyz=0 0 0 rpy=2.46519e-32 -8.59206e-33 -3.9443e-31; parent dm_j4340_motor_1 -> dm_j10010l_side_cover
- joint group_1_fastened_joint_5: child dm_j4340_controller_cover_5 -> dm_j4340_controller_cover_9; origin xyz=0 -0.00025 0 rpy=-5.8789e-32 0 0 -> xyz=0 -0.00175 0 rpy=-9.86076e-32 7.88861e-31 1.54465e-37; parent dm_j4340_motor_5 -> dm_j4340_motor_9
- joint group_1_fastened_joint_6: child dm_j10010l_stator__1__2 -> dm_j4340_controller_cover_3; origin xyz=-1.73472e-18 0.0659355 5.55112e-17 rpy=1.2326e-32 1.70026e-74 -2.75883e-42 -> xyz=-2.77556e-17 -0.00175 -5.55112e-17 rpy=3.34096e-52 -9.86076e-32 -6.77626e-21; parent dm_j10010l_rotor_8 -> dm_j4340_motor_3
- joint group_1_fastened_joint_7: axis -0 -0 -1 -> 0 0 1; child dm_j10010l_side_cover_8 -> dm_j4340_controller_cover_2; origin xyz=-1.73472e-18 0.0659355 5.55112e-17 rpy=1.2326e-32 1.70026e-74 -2.75883e-42 -> xyz=-2.77556e-17 0 6.93889e-18 rpy=-7.88861e-31 -1.97215e-31 6.77626e-21; parent dm_j10010l_rotor_8 -> dm_j4340_motor_2
- joint group_1_fastened_joint_8: axis -0 -0 -1 -> 0 0 1; child dm_j10010l_controller_cover_8 -> dm_j4340_controller_cover_13; origin xyz=-1.73472e-18 -3.46945e-18 5.55112e-17 rpy=1.2326e-32 1.70026e-74 -2.75883e-42 -> xyz=0 -0.00025 0 rpy=-5.8789e-32 0 0; parent dm_j10010l_side_cover_8 -> dm_j4340_motor_13
- joint group_1_fastened_joint_9: child dm_j4340_controller_cover_4 -> dm_j10010l_stator__1__2; origin xyz=1.11022e-16 -0.00025 0 rpy=1.50704e-32 -0 0 -> xyz=-1.73472e-18 0.0659355 5.55112e-17 rpy=1.2326e-32 1.70026e-74 -2.75883e-42; parent dm_j4340_motor_4 -> dm_j10010l_rotor_2
- joint left_ankle_pitch_joint: limit lower=-0.6 upper=0.6 effort=1 velocity=1 -> lower=-0.6 upper=0.6 effort=27 velocity=8
- joint left_ankle_roll_joint: limit lower=-0.5 upper=0.5 effort=1 velocity=1 -> lower=-0.5 upper=0.5 effort=27 velocity=8
- joint left_hip_pitch_joint: limit lower=-0.698132 upper=2.0944 effort=1 velocity=1 -> lower=-2.094 upper=0.7854 effort=120 velocity=25; parent dm_j10010l_rotor_4 -> dm_j10010l_rotor_5
- joint left_hip_roll_joint: limit lower=-0.999829 upper=0.199997 effort=1 velocity=1 -> lower=-0.2 upper=1 effort=120 velocity=25; parent dm_j10010l_rotor_6 -> dm_j10010l_rotor_7
- joint left_hip_yaw_joint: limit lower=-0.199997 upper=1 effort=1 velocity=1 -> lower=-1 upper=0.2 effort=120 velocity=25; parent dm_j10010l_rotor_7 -> dm_j10010l_rotor_8
- joint left_knee_joint: limit lower=-0.2 upper=2.5 effort=1 velocity=1 -> lower=-0.2 upper=2.5 effort=120 velocity=25
- joint mate_connector_1: child mate_connector_1 -> mate_connector_1_1
- joint mate_connector_1_1: child mate_connector_1_1 -> mate_connector_1
- joint right_ankle_pitch_joint: limit lower=-0.6 upper=0.6 effort=1 velocity=1 -> lower=-0.6 upper=0.6 effort=27 velocity=8
- joint right_ankle_roll_joint: limit lower=-0.5 upper=0.5 effort=1 velocity=1 -> lower=-0.5 upper=0.5 effort=27 velocity=8
- joint right_hip_pitch_joint: limit lower=-0.174533 upper=2.26893 effort=1 velocity=1 -> lower=-2.094 upper=0.7854 effort=120 velocity=25; parent dm_j10010l_rotor_2 -> dm_j10010l_rotor_3
- joint right_hip_roll_joint: limit lower=-0.199997 upper=1 effort=1 velocity=1 -> lower=-1 upper=0.2 effort=120 velocity=25
- joint right_hip_yaw_joint: limit lower=-0.199997 upper=1 effort=1 velocity=1 -> lower=-0.2 upper=1 effort=120 velocity=25
- joint right_knee_joint: limit lower=-0.2 upper=2.5 effort=1 velocity=1 -> lower=-0.2 upper=2.5 effort=120 velocity=25; parent dm_j10010l_stator__1__4 -> dm_j10010l_stator__1__1
- joint waist_yaw: limit lower=-3.14159 upper=3.14159 effort=1 velocity=1 -> lower=-3.14 upper=3.14 effort=120 velocity=25; origin xyz=-3.46945e-18 -0.0659355 -5.89019e-21 rpy=1.5708 8.08706e-16 -9.45117e-16 -> xyz=-1.04083e-17 -0.0659355 -3.26795e-18 rpy=1.5708 6.57474e-16 -8.14127e-16
